File: anotterwatch.kicad_pcb (KiCad board)
At the start: 2 copper layers, 48.5 x 43 mm, 82 parts, among them J1 USB_C_Receptacle_USB2.0, J2 Conn_01x05, Q1 Q_NMOS_GSD, Q2 nfet, Q3 npn, Q4 npn, Q5 2N7002, Q6 2N7002, U1 USBLC6-4SC6, U10 TS5A2053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

Commit message: ADD: Jog switch
Parts:
- removed D3: LED, badgelib:RZX-S020CCW-0.4T
- added REF**: TMHU26, badgelib:TMHU26, B.Cu at (121.7, 81.5)
- moved J1 2.29 mm to (112.1, 75.9)
- moved U3 1.90 mm to (111.0, 81.0)
Changed lines of the file:
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@@
   )
   (module Package_SO:SOIC-16_3.9x9.9mm_P1.27mm (layer B.Cu)
-    (at 111.887 82.677 270)
+    (at 111 81 270)
     (descr "16-Lead Plastic Small Outline (SL) - Narrow, 3.90 mm Body [SOIC] (see Microchip Packaging Specification 00000049BS.pdf)")
     (tags "SOIC 1.27")
@@
     )
   )
-  (module badgelib:RZX-S020CCW-0.4T (layer B.Cu)
-    (at 120.457661 127.223766)
-    (fp_text reference D3 (at 0 1.25) (layer B.SilkS)
-      (effects (font (size 1 1) (thickness 0.15)) (justify mirror))
-    )
-    (fp_text value LED (at 0 2.75) (layer B.Fab)
-      (effects (font (size 1 1) (thickness 0.15)) (justify mirror))
-    )
-    (fp_line (start -1.75 -0.75) (end 1.75 -0.75) (layer B.SilkS) (width 0.15))
-    (fp_line (start 1.75 -0.75) (end 1.75 -0.5) (layer B.SilkS) (width 0.15))
-    (fp_line (start -1.75 -0.75) (end -1.75 -0.5) (layer B.SilkS) (width 0.15))
-    (fp_line (start -1 0.25) (end 1 0.25) (layer B.SilkS) (width 0.15))
-    (pad K smd rect (at -1.7 0) (size 1.2 0.7) (layers B.Cu B.Paste B.Mask))
-    (pad A smd rect (at 1.7 0) (size 1.2 0.7) (layers B.Cu B.Paste B.Mask))
-  )
   (module badgelib:ST7789V (layer B.Cu)
     (at 86.614 96.774 90)
@@
   )
   (module "badgelib:USB-C 16Pin" (layer B.Cu)
-    (at 114.427 75.819)
+    (at 112.141 75.946)
     (fp_text reference J1 (at 0 -1.5) (layer B.SilkS)
       (effects (font (size 1 1) (thickness 0.15)) (justify mirror))
@@
     (pad 1 np_thru_hole circle (at 0 0) (size 2.2 2.2) (drill 2.2) (layers *.Cu *.Mask))
   )
+  (module badgelib:TMHU26 (layer B.Cu)
+    (at 121.666 81.534 90)
+    (fp_text reference REF** (at 0 -5.75 90) (layer B.SilkS)
+      (effects (font (size 1 1) (thickness 0.15)) (justify mirror))
+    )
+    (fp_text value TMHU26 (at 0 1.75 90) (layer B.Fab)
+      (effects (font (size 1 1) (thickness 0.15)) (justify mirror))
+    )
+    (fp_line (start -2.5 4.5) (end 2.5 4.5) (layer B.SilkS) (width 0.15))
+    (fp_line (start -6 3.75) (end -6 2.5) (layer B.SilkS) (width 0.15))
+    (fp_line (start 6 3.75) (end 6 2.5) (layer B.SilkS) (width 0.15))
+    (fp_line (start -2.5 4.5) (end -6 3.75) (layer B.SilkS) (width 0.15))
+    (fp_line (start 6 3.75) (end 2.5 4.5) (layer B.SilkS) (width 0.15))
+    (fp_line (start 6 -4.25) (end 3.75 -4.25) (layer B.SilkS) (width 0.15))
+    (fp_line (start -6 -4.25) (end -3.75 -4.25) (layer B.SilkS) (width 0.15))
+    (fp_line (start -6 -4.25) (end -6 0.25) (layer B.SilkS) (width 0.15))
+    (fp_line (start 6 0.25) (end 6 -4.25) (layer B.SilkS) (width 0.15))
+    (fp_text user "Board Edge" (at 0 5.75 90) (layer Eco1.User)
+      (effects (font (size 1 1) (thickness 0.15)))
+    )
+    (fp_line (start -4 4.8) (end 4 4.8) (layer Eco1.User) (width 0.15))
+    (pad 4 smd rect (at -5.2 1.3 90) (size 1.8 1.7) (layers B.Cu B.Paste B.Mask))
+    (pad 3 smd rect (at 5.2 1.3 90) (size 1.8 1.7) (layers B.Cu B.Paste B.Mask))
+    (pad 2 smd rect (at 2.5 -3.55 90) (size 1.9 1.8) (layers B.Cu B.Paste B.Mask))
+    (pad T smd rect (at 0 -3.55 90) (size 1.9 1.8) (layers B.Cu B.Paste B.Mask))
+    (pad 1 smd rect (at -2.5 -3.55 90) (size 1.9 1.8) (layers B.Cu B.Paste B.Mask))
+    (pad "" np_thru_hole circle (at 2.5 0.2 90) (size 1.1 1.1) (drill 1.1) (layers *.Cu *.Mask))
+    (pad "" np_thru_hole circle (at -2.5 0.2 90) (size 1.1 1.1) (drill 1.1) (layers *.Cu *.Mask))
+  )
   (dimension 48.5 (width 0.3) (layer Eco2.User)
