File: anotterwatch.kicad_pcb (KiCad board)
At the start: 2 copper layers, 48.5 x 43 mm, 121 parts, among them J1 Conn_02x02_Odd_Even, J2 Micro_SD_Card, J3 Conn_01x05, J4 USB_C_Receptacle_USB2.0, Q1 AO3400, Q10 Q_PMOS_GDS, Q2 AO3400, Q3 AO3400, Q4 AO3400, Q5 AO3400, Q6 2N7002, Q7 2N7002, Q8 2N7002, Q9 2N7002, SW1 SW_SPST, U1 BMI270, U10 TS5A2053, U11 TS5A2053, U12 ADS7946SRTET, U13 TP4056, U14 TPS63001DRCR, U2 CH340C, U3 ESP32, U4 ST7789V, U5 REF2915, U6 TCA9535MRGER, U7 TLV9062S, U8 OPA2322S, U9 USBLC6-4SC6

Commit message: ADD:started to place footprints
Parts:
- removed D7: D_Small, Diode_SMD:D_SMA
- added C31: 100n, Capacitor_SMD:C_0402_1005Metric, B.Cu at (113.9, 109.3)
- added C32: 100n, Capacitor_SMD:C_0402_1005Metric, B.Cu at (86.9, 74.8)
- added C33: 100n, Capacitor_SMD:C_0402_1005Metric, B.Cu at (117.1, 75.7)
- added C34: 100n, Capacitor_SMD:C_0402_1005Metric, B.Cu at (85.7, 106.4)
- added D5: LED, badgelib:RZX-S020CCW-0.4T, B.Cu at (96.0, 75.5)
- added D6: D_Small, Diode_SMD:D_SOD-123F, B.Cu at (81.2, 81.7)
- added LS1: Speaker, Connector_Molex:Molex_KK-254_AE-6410-02A_1x02_P2.54mm_Vertical, F.Cu at (176.4, 77.4)
- added R48: 5k1, Resistor_SMD:R_0402_1005Metric, B.Cu at (87.1, 77.2)
- added R49: 5k1, Resistor_SMD:R_0402_1005Metric, B.Cu at (87.1, 76.3)
- added R50: 47k, Resistor_SMD:R_0402_1005Metric, B.Cu at (85.3, 74.5)
- added R51: 100, Resistor_SMD:R_0402_1005Metric, B.Cu at (78.6, 91.6)
- C1, C10, C11, C12, C13, C14, C16, C17, C18, C19, C2, C20, C21, C22, C24, C28, C29, C4, C5, C6, C7, C8, C9: footprint Capacitor_SMD:C_0603_1608Metric -> Capacitor_SMD:C_0402_1005Metric
- D1, D2, D3, D4: footprint LED_SMD:LED_SK6812MINI_PLCC4_3.5x3.5mm_P1.75mm -> badgelib:LED_SK6812MINI_PLCC4_3.5x3.5mm_P1.75mm
- J2: renamed from J1; value Conn_02x02_Odd_Even -> Shitty Add-On
- Q10: value Q_PMOS_GDS -> Q_PMOS_GSD
- Q4: value AO3400 -> Q_PMOS_GSD
- Q6, Q7, Q8, Q9: value 2N7002 -> AO3400
- R1: value 5k1 -> 47k; footprint Resistor_SMD:R_0603_1608Metric -> Resistor_SMD:R_0402_1005Metric
- R10: value 47k -> 100; footprint Resistor_SMD:R_0603_1608Metric -> Resistor_SMD:R_0402_1005Metric
- R11, R18: value 10 -> 47k; footprint Resistor_SMD:R_0603_1608Metric -> Resistor_SMD:R_0402_1005Metric
- R12, R22: value 100 -> 47k; footprint Resistor_SMD:R_0603_1608Metric -> Resistor_SMD:R_0402_1005Metric
- R14: value 47k -> 10
- R16, R20, R46, R8: value 47k -> 5k1; footprint Resistor_SMD:R_0603_1608Metric -> Resistor_SMD:R_0402_1005Metric
- R17, R19, R27, R28, R3, R4, R45, R5, R6, R7: footprint Resistor_SMD:R_0603_1608Metric -> Resistor_SMD:R_0402_1005Metric
- R2, R9: value 5k1 -> 10
- R21: value 680 -> 5k1; footprint Resistor_SMD:R_0603_1608Metric -> Resistor_SMD:R_0402_1005Metric
- R23: value 390k -> 47k; footprint Resistor_SMD:R_0603_1608Metric -> Resistor_SMD:R_0402_1005Metric
- R24: value 680 -> 47k; footprint Resistor_SMD:R_0603_1608Metric -> Resistor_SMD:R_0402_1005Metric
- R25: value 390k -> 680; footprint Resistor_SMD:R_0603_1608Metric -> Resistor_SMD:R_0402_1005Metric
- R26: value 390k -> 100; footprint Resistor_SMD:R_0603_1608Metric -> Resistor_SMD:R_0402_1005Metric
- R29, R30, R31, R39: value 10M -> 390k; footprint Resistor_SMD:R_0603_1608Metric -> Resistor_SMD:R_0402_1005Metric
- R32: value 10M -> 680; footprint Resistor_SMD:R_0603_1608Metric -> Resistor_SMD:R_0402_1005Metric
- R33, R34, R35: value 390k -> 10M
- R36: value 47k -> 10M
- R37, R38: value 2M2 -> 390k; footprint Resistor_SMD:R_0603_1608Metric -> Resistor_SMD:R_0402_1005Metric
- R40: value 10M -> 47k; footprint Resistor_SMD:R_0603_1608Metric -> Resistor_SMD:R_0402_1005Metric
- R41, R42: value 5k1 -> 2M2; footprint Resistor_SMD:R_0603_1608Metric -> Resistor_SMD:R_0402_1005Metric
- R43: value 390k -> 10M; footprint Resistor_SMD:R_0603_1608Metric -> Resistor_SMD:R_0402_1005Metric
- R44: value 5k1 -> 10M; footprint Resistor_SMD:R_0603_1608Metric -> Resistor_SMD:R_0402_1005Metric
- R47: value 100 -> 390k; footprint Resistor_SMD:R_0603_1608Metric -> Resistor_SMD:R_0402_1005Metric
- U1: value BMI270 -> ST7789V; footprint badgelib:BMI270 -> badgelib:ST7789V
- U4: value ST7789V -> BMI270; footprint badgelib:ST7789V -> badgelib:BMI270
- moved C2 131.0 mm to (74.9, 96.8)
- moved C4 131.0 mm to (74.9, 95.3)
- moved C5 131.0 mm to (71.7, 92.9)
- moved R10 131.0 mm to (74.7, 92.3)
- moved R17 131.0 mm to (74.3, 88.4)
- moved R3 131.0 mm to (74.3, 89.9)
- moved R6 131.0 mm to (74.7, 93.8)
- moved R8 131.0 mm to (71.3, 88.2)
- moved C30 129.2 mm to (79.1, 85.0), turned to 90 degrees
- moved R7 129.1 mm to (71.9, 90.0)
- moved Q10 127.7 mm to (80.0, 92.9), turned to 180 degrees
- moved C28 125.3 mm to (78.6, 89.8), turned to 90 degrees
- moved U14 123.5 mm to (80.9, 88.5), turned to 270 degrees
- moved C27 120.0 mm to (82.4, 94.6), turned to 90 degrees
- moved L2 119.8 mm to (81.5, 84.5)
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- renumbered J2 to J1
Connections:
- C1 pad 1: VBUS -> Net-(C1-Pad1)
- C2 pad 1: Net-(C2-Pad1) -> IPS_RST
- C8 pad 1: IPS_RST -> BTN_UP
- D1 pad 2: Net-(D1-Pad2) -> GND
- D1 pad 4: +3V3 -> Net-(C31-Pad2)
- D2 pad 2: Net-(D1-Pad2) -> GND
- D2 pad 4: +3V3 -> Net-(C31-Pad2)
- D3 pad 2: Net-(D1-Pad2) -> GND
- D3 pad 4: +3V3 -> Net-(C31-Pad2)
- D4 pad 2: Net-(D1-Pad2) -> GND
- D4 pad 4: +3V3 -> Net-(C31-Pad2)
- J1 pad 5: Net-(J2-Pad5) -> Net-(J1-Pad5)
- J1 pad 7: Net-(J2-Pad7) -> Net-(J1-Pad7)
- Q3 pad 1: PARTY_ENABLE -> IPS_LED
- Q3 pad 3: Net-(D1-Pad2) -> Net-(Q3-Pad3)
- Q4 pad 1: IPS_LED -> PARTY_ENABLE
- Q4 pad 2: GND -> +3V3
- Q4 pad 3: Net-(Q4-Pad3) -> Net-(C31-Pad2)
- Q5 pad 1: WHITE_LED -> Net-(Q5-Pad1)
- Q5 pad 2: GND -> Net-(Q5-Pad2)
- R1 pad 1: I2C_SDA -> +3V3
- R1 pad 2: +3V3 -> IPS_RST
- R10 pad 1: +3V3 -> Net-(J1-Pad7)
- R10 pad 2: BTN_CNTR -> SD_DATA0
- R11 pad 1: Net-(J2-Pad5) -> Net-(Q5-Pad1)
- R11 pad 2: SD_CLK -> WHITE_LED
- R12 pad 1: Net-(J2-Pad7) -> Net-(Q5-Pad1)
- R12 pad 2: SD_DATA0 -> GND
- R14 pad 1: PARTY_ENABLE -> Net-(Q5-Pad2)
- R15 pad 1: +BATT -> Net-(Q5-Pad2)
- R15 pad 2: Net-(D5-Pad2) -> GND
- R16 pad 1: WHITE_LED -> +BATT
- R16 pad 2: GND -> BTN_UP
- R17 pad 1: +3V3 -> BTN_UP
- R17 pad 2: IPS_RST -> GND
- R18 pad 1: +BATT -> +3V3
- R18 pad 2: Net-(D6-Pad2) -> BTN_DOWN
- R19 pad 1: ESP32_DAC -> +3V3
- R19 pad 2: ADC_REF -> BTN_CNTR
- R2 pad 1: +3V3 -> Net-(Q3-Pad3)
- R2 pad 2: I2C_SCL -> Net-(R2-Pad2)
- R20 pad 1: GNDA -> I2C_SDA
- R20 pad 2: ESP32_DAC -> +3V3
- R21 pad 1: Net-(J3-Pad3) -> +3V3
- R21 pad 2: Net-(R21-Pad2) -> I2C_SCL
- R22 pad 1: Net-(J3-Pad3) -> ESP32_DAC
- R22 pad 2: Net-(C15-Pad1) -> ADC_REF
- R23 pad 1: Net-(J3-Pad3) -> GNDA
- R23 pad 2: Net-(R23-Pad2) -> ESP32_DAC
- R24 pad 1: Net-(J3-Pad2) -> Net-(C15-Pad2)
- R24 pad 2: Net-(R24-Pad2) -> Net-(C15-Pad1)
- R25 pad 1: Net-(J3-Pad2) -> Net-(J3-Pad3)
- R26 pad 1: Net-(C17-Pad1) -> Net-(J3-Pad3)
- R26 pad 2: ADC_REF -> Net-(C15-Pad1)
- R27 pad 1: Net-(C18-Pad1) -> Net-(J3-Pad3)
- R27 pad 2: ADC_REF -> Net-(R27-Pad2)
- R28 pad 1: Net-(J3-Pad1) -> Net-(J3-Pad2)
- R29 pad 1: Net-(J3-Pad1) -> Net-(J3-Pad2)
- R29 pad 2: PROBE1 -> Net-(R29-Pad2)
- R3 pad 2: SD_DATA0 -> IO0
- R30 pad 1: Net-(J3-Pad2) -> Net-(C17-Pad1)
- R30 pad 2: PROBE2 -> ADC_REF
- R31 pad 1: Net-(J3-Pad4) -> Net-(C18-Pad1)
- R31 pad 2: PROBE1 -> ADC_REF
- R32 pad 1: Net-(J3-Pad5) -> Net-(J3-Pad1)
- R32 pad 2: PROBE2 -> Net-(R32-Pad2)
- R33 pad 1: GNDA -> Net-(J3-Pad1)
- R33 pad 2: Net-(C17-Pad1) -> PROBE1
- R34 pad 1: GNDA -> Net-(J3-Pad2)
- R34 pad 2: Net-(C18-Pad1) -> PROBE2
- R35 pad 1: Net-(J3-Pad1) -> Net-(J3-Pad4)
- R35 pad 2: Net-(R35-Pad2) -> PROBE1
- R36 pad 1: ADC_ENABLE -> Net-(J3-Pad5)
- R36 pad 2: +3V3 -> PROBE2
- R37 pad 1: PROBE1 -> GNDA
- R37 pad 2: Net-(C19-Pad1) -> Net-(C17-Pad1)
- R38 pad 1: PROBE2 -> GNDA
- R38 pad 2: Net-(C20-Pad1) -> Net-(C18-Pad1)
- R39 pad 1: Net-(C21-Pad2) -> Net-(J3-Pad1)
- R39 pad 2: PROBE1 -> Net-(R39-Pad2)
- R4 pad 2: IO0 -> EN
- R40 pad 1: Net-(C22-Pad2) -> ADC_ENABLE
- R40 pad 2: PROBE2 -> +3V3
- R41 pad 1: GND -> PROBE1
- R41 pad 2: Net-(J4-PadA5) -> Net-(C19-Pad1)
- R42 pad 1: GND -> PROBE2
- R42 pad 2: Net-(J4-PadB5) -> Net-(C20-Pad1)
- R43 pad 1: +3V3 -> Net-(C21-Pad2)
- R43 pad 2: CHRG -> PROBE1
- R44 pad 1: Net-(R44-Pad1) -> Net-(C22-Pad2)
- R44 pad 2: GND -> PROBE2
- R45 pad 1: Net-(R44-Pad1) -> GND
- R45 pad 2: GND -> Net-(J4-PadA5)
- R46 pad 1: VBUS -> GND
- R46 pad 2: GND -> Net-(J4-PadB5)
- R47 pad 1: +BATT -> +3V3
- R47 pad 2: Net-(C28-Pad1) -> CHRG
- R5 pad 2: BTN_UP -> SD_DATA0
- R7 pad 2: EN -> PARTY_ENABLE
- R8 pad 2: BTN_DOWN -> SD_CMD
- R9 pad 1: +3V3 -> Net-(J1-Pad5)
- R9 pad 2: SD_CMD -> SD_CLK
- U1 pad 10: Net-(U1-Pad10) -> IPS_MOSI
- U1 pad 11: Net-(U1-Pad11) -> IPS_RST
- U1 pad 2: Net-(U1-Pad2) -> Net-(R2-Pad2)
- U1 pad 3: Net-(U1-Pad3) -> +3V3
- U1 pad 4: WAKE1 -> +3V3
- U1 pad 5: +3V3 -> GND
- U1 pad 7: GND -> IPS_DC
- U1 pad 8: +3V3 -> GND
- U1 pad 9: Net-(U1-Pad9) -> +3V3
- U13 pad 2: Net-(R44-Pad1) -> Net-(R48-Pad1)
- U2 pad 4: Net-(C2-Pad1) -> Net-(C1-Pad1)
- U4 pad 10: IPS_MOSI -> Net-(U4-Pad10)
- U4 pad 11: IPS_RST -> Net-(U4-Pad11)
- U4 pad 12: (no net) -> +3V3
- U4 pad 2: Net-(Q4-Pad3) -> Net-(U4-Pad2)
- U4 pad 3: +3V3 -> Net-(U4-Pad3)
- U4 pad 4: +3V3 -> WAKE1
- U4 pad 5: GND -> +3V3
- U4 pad 7: IPS_DC -> GND
- U4 pad 8: GND -> +3V3
- U4 pad 9: +3V3 -> Net-(U4-Pad9)
- U6 pad 10: Net-(R28-Pad2) -> Net-(R32-Pad2)
- U6 pad 12: Net-(R25-Pad2) -> Net-(R29-Pad2)
- U6 pad 13: Net-(R24-Pad2) -> Net-(R28-Pad2)
- U6 pad 15: Net-(R23-Pad2) -> Net-(R27-Pad2)
- U6 pad 16: Net-(R21-Pad2) -> Net-(R25-Pad2)
- U6 pad 8: Net-(R35-Pad2) -> Net-(R39-Pad2)
- U9 pad 3: PROBE2 -> PROBE1
- U9 pad 4: PROBE1 -> PROBE2
Routing:
- net PROBE2: track 0.00 -> 21.0 mm
- net Net-(J3-Pad2): track 0.00 -> 17.7 mm
- net PROBE1: track 0.00 -> 17.3 mm
- net ADC_REF: track 0.00 -> 5.99 mm
- net ESP32_DAC: track 0.00 -> 5.83 mm
- net Net-(C18-Pad1): track 0.00 -> 5.07 mm
- net Net-(J3-Pad5): track 0.00 -> 4.97 mm
- net Net-(C19-Pad1): track 0.00 -> 3.95 mm
- net Net-(U12-Pad8): track 0.00 -> 3.44 mm
- net Net-(C21-Pad2): track 0.00 -> 3.27 mm
- net Net-(C17-Pad1): track 0.00 -> 2.70 mm
- net Net-(J3-Pad1): track 0.00 -> 2.06 mm
- net Net-(U12-Pad5): track 0.00 -> 2.04 mm
- net Net-(C22-Pad2): track 0.00 -> 1.85 mm
- net Net-(C20-Pad1): track 0.00 -> 1.82 mm
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Other:
- copper layers 2 -> 4
- net class Default: clearance 0.2 -> 0.127; trace_width 0.25 -> 0.15; via_dia 0.8 -> 0.6; via_drill 0.4 -> 0.3
- net class HV added: clearance 0.127, trace_width 0.15, via_dia 0.6, via_drill 0.3
- rule trace_clearance: 0.2 -> 0.127
- rule trace_min: 0.2 -> 0.15
- rule via_min_size: 0.4 -> 0.6
- board text added: "IPS FFC"

Commit message: ADD: started routing
Parts:
- added C35: 470p, Capacitor_SMD:C_0402_1005Metric, B.Cu at (113.1, 88.7)
- added C36: 470p, Capacitor_SMD:C_0402_1005Metric, B.Cu at (111.9, 90.0)
- added R52: 10, Resistor_SMD:R_0603_1608Metric, B.Cu at (114.2, 90.2)
- added R53: 10, Resistor_SMD:R_0603_1608Metric, B.Cu at (113.3, 91.1)
- U7, U8: footprint Package_SON:VSON-10-1EP_3x3mm_P0.5mm_EP1.2x2mm -> badgelib:VSSOP-10
- moved R3 29.5 mm to (102.5, 81.1), turned to 270 degrees
- moved C4 29.3 mm to (97.5, 76.7), turned to 90 degrees
- moved R10 26.9 mm to (99.5, 81.6), turned to 90 degrees
- moved R7 26.7 mm to (98.6, 89.6), turned to 270 degrees
- moved C13 26.5 mm to (107.9, 85.4), turned to 90 degrees
- moved R8 26.4 mm to (97.3, 83.8), turned to 270 degrees
- moved R6 26.0 mm to (98.8, 83.8), turned to 270 degrees
- moved R17 25.0 mm to (96.2, 76.3)
- moved C2 23.3 mm to (97.2, 90.2), turned to 90 degrees
- moved R50 17.1 mm to (80.8, 91.0)
- moved R19 15.3 mm to (101.1, 81.3), turned to 180 degrees
- moved R18 15.2 mm to (101.1, 80.5), turned to 180 degrees
- moved R20 12.7 mm to (88.0, 83.3), turned to 270 degrees
- moved R21 12.7 mm to (88.9, 83.3), turned to 90 degrees
- moved U4 11.7 mm to (89.7, 86.2), turned to 180 degrees
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Connections:
- U12 pad 5: Net-(U12-Pad5) -> Net-(C35-Pad1)
- U12 pad 8: Net-(U12-Pad8) -> Net-(C36-Pad2)
- U8 pad 1: Net-(U12-Pad5) -> Net-(R52-Pad2)
- U8 pad 2: Net-(U12-Pad5) -> Net-(R52-Pad2)
- U8 pad 8: Net-(U12-Pad8) -> Net-(R53-Pad2)
- U8 pad 9: Net-(U12-Pad8) -> Net-(R53-Pad2)
Routing:
- net SE_ENABLE: track 0.00 -> 50.3 mm, vias 0 -> 3
- net AFE_ENABLE: track 0.00 -> 37.5 mm, vias 0 -> 5
- net Net-(J1-Pad5): track 0.00 -> 33.8 mm, vias 0 -> 2
- net Net-(J1-Pad7): track 0.00 -> 33.4 mm, vias 0 -> 2
- net Net-(J3-Pad1): track 2.06 -> 34.3 mm, vias 0 -> 3
- net SD_DATA3: track 0.00 -> 31.8 mm, vias 0 -> 3
- net SD_DATA1: track 0.00 -> 31.8 mm, vias 0 -> 2
- net MUX_ENABLE: track 0.00 -> 31.2 mm, vias 0 -> 3
- net SD_CMD: track 0.00 -> 30.4 mm, vias 0 -> 3
- net Net-(J3-Pad3): track 0.00 -> 30.1 mm, vias 0 -> 2
- net SD_DATA2: track 0.00 -> 29.7 mm, vias 0 -> 2
- net MUX_CH2: track 0.00 -> 28.6 mm, vias 0 -> 2
- net ADC_MISO: track 0.00 -> 25.8 mm, vias 0 -> 2
- net Net-(J3-Pad2): track 17.7 -> 39.4 mm, vias 0 -> 2
- net ADC_CS: track 0.00 -> 19.3 mm, vias 0 -> 2
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
Commit message: ADD: tbc
Parts:
- moved R13 0.30 mm to (93.0, 85.6)
- moved Q5 0.23 mm to (99.6, 76.6)
Routing:
- net IPS_LED: track 0.00 -> 31.1 mm, vias 0 -> 2
- net IPS_DC: track 0.00 -> 24.8 mm, vias 0 -> 2
- net ADC_CH_SEL: track 0.91 -> 21.2 mm, vias 1 -> 2
- net Net-(R2-Pad2): track 0.00 -> 5.48 mm
- net ESP32_DAC: track 7.23 -> 10.8 mm, vias 0 -> 1
- net Net-(Q3-Pad3): track 0.00 -> 1.48 mm
- net ADC_SCK: track 16.5 -> 17.8 mm, vias 2 -> 3
- net Net-(R13-Pad2): track 1.64 -> 2.35 mm

Commit message: added pwoer layout
Parts:
- moved R45 0.95 mm to (105.8, 75.7)
- moved R46 0.87 mm to (104.8, 75.7)
- moved C32 0.67 mm to (86.5, 74.3), turned to 180 degrees
- turned C5 to 270 degrees
Connections:
- C32 pad 2: Net-(C32-Pad2) -> Net-(C31-Pad2)
- U1 pad 9: +3V3 -> ADC_SCK
- U7 pad 8: ESP32_ADC -> ESP_ADC
- U7 pad 9: ESP32_ADC -> ESP_ADC
Routing:
- net Net-(BT1-Pad1): track 18.1 -> 43.5 mm, vias 0 -> 2
- net GND: track 0.00 -> 25.2 mm, vias 0 -> 12
- net +3V3: track 4.26 -> 28.5 mm, vias 0 -> 2
- net VBUS: track 0.00 -> 24.2 mm, vias 0 -> 2
- net Net-(Q10-Pad2): track 0.00 -> 8.32 mm
- net Net-(C28-Pad1): track 0.00 -> 6.37 mm, vias 0 -> 2
- net CHRG: track 0.00 -> 4.38 mm
- net Net-(J4-PadB5): track 7.22 -> 11.5 mm
- net Net-(R48-Pad1): track 0.00 -> 2.37 mm
- net +BATT: track 0.00 -> 1.20 mm, vias 0 -> 7
- net Net-(J4-PadA5): track 9.01 -> 8.25 mm
- net ESP_ADC: track 0.00 -> 0.55 mm
- net ESP32_ADC: track 0.55 -> 0.00 mm
- net (no net): vias 0 -> 2
- added copper zone on B.Cu, net +3V3
- added copper zone on B.Cu, net +BATT
- added copper zone on In2.Cu, net +BATT
- added copper zone on B.Cu, net GND
- added copper zone on B.Cu, net Net-(L2-Pad1)
- added copper zone on B.Cu, net Net-(L2-Pad2)
- added copper zone on B.Cu, net VBUS

Commit message: fixed 3D models
Parts:
- removed D6: D_Small, Diode_SMD:D_SOD-123F
- removed Q10: Q_PMOS_GSD, Package_TO_SOT_SMD:SOT-23
- removed R50: 47k, Resistor_SMD:R_0402_1005Metric
- BT1: footprint Connector_JST:JST_GH_BM02B-GHS-TBT_1x02-1MP_P1.25mm_Vertical -> badgelib:JST_GH_BM02B-GHS-TBT_1x02-1MP_P1.25mm_Vertical
- J1: footprint ST-TF-003A:SUNTECH_ST-TF-003A -> badgelib:SUNTECH_ST-TF-003A
- Q4: value Q_PMOS_GSD -> AO3400
- R48, R49: value 5k1 -> 680
Connections:
- C31 pad 1: GND -> Net-(C31-Pad1)
- C31 pad 2: Net-(C31-Pad2) -> +3V3
- C32 pad 1: GND -> Net-(C31-Pad1)
- C32 pad 2: Net-(C31-Pad2) -> +3V3
- C33 pad 1: GND -> Net-(C31-Pad1)
- C33 pad 2: Net-(C31-Pad2) -> +3V3
- C34 pad 1: GND -> Net-(C31-Pad1)
- C34 pad 2: Net-(C31-Pad2) -> +3V3
- D1 pad 2: GND -> Net-(C31-Pad1)
- D1 pad 4: Net-(C31-Pad2) -> +3V3
- D2 pad 2: GND -> Net-(C31-Pad1)
- D2 pad 4: Net-(C31-Pad2) -> +3V3
- D3 pad 2: GND -> Net-(C31-Pad1)
- D3 pad 4: Net-(C31-Pad2) -> +3V3
- D4 pad 2: GND -> Net-(C31-Pad1)
- D4 pad 4: Net-(C31-Pad2) -> +3V3
- Q4 pad 2: +3V3 -> GND
- Q4 pad 3: Net-(C31-Pad2) -> Net-(C31-Pad1)
- R48 pad 2: GND -> Net-(R48-Pad2)
- R49 pad 1: Net-(R48-Pad1) -> GND
- R49 pad 2: GND -> Net-(R48-Pad1)
- R7 pad 1: +3V3 -> PARTY_ENABLE
- R7 pad 2: PARTY_ENABLE -> GND
- SW1 pad 2: Net-(Q10-Pad2) -> +BATT
- U13 pad 2: Net-(R48-Pad1) -> Net-(R48-Pad2)
Routing:
- net VBUS: track 24.2 -> 7.18 mm, vias 2 -> 0
- net +BATT: track 1.20 -> 11.2 mm, vias 7 -> 6
- net Net-(Q10-Pad2): track 8.32 -> 0.00 mm
- net +3V3: track 28.5 -> 25.8 mm
- net GND: vias 12 -> 11
