File: anotterwatch.sch (KiCad schematic (older format))
At the start: 27 parts, among them J1 USB_C_Receptacle_USB2.0, Q1 Q_NMOS_GSD, U1 USBLC6-4SC6

Commit message: added datasheet esp
Connections:
- wire segments 59 -> 71
Changed lines of the file:
@@
 	1    0    0    -1
 $EndComp
+$Comp
+L power:VCC #PWR?
+U 1 1 5C71EB10
+P 4050 1900
+F 0 "#PWR?" H 4050 1750 50  0001 C CNN
+F 1 "VCC" H 4067 2073 50  0000 C CNN
+F 2 "" H 4050 1900 50  0001 C CNN
+F 3 "" H 4050 1900 50  0001 C CNN
+	1    4050 1900
+	1    0    0    -1
+$EndComp
+Wire Wire Line
+	4200 1950 4050 1950
+Wire Wire Line
+	4050 1950 4050 1900
+Wire Wire Line
+	4200 2050 4050 2050
+Wire Wire Line
+	4050 2050 4050 1950
+Connection ~ 4050 1950
+Wire Wire Line
+	4200 2150 4050 2150
+Wire Wire Line
+	4050 2150 4050 2050
+Connection ~ 4050 2050
+Wire Wire Line
+	4200 2250 4050 2250
+Wire Wire Line
+	4050 2250 4050 2150
+Connection ~ 4050 2150
+Wire Wire Line
+	4200 2350 4050 2350
+Wire Wire Line
+	4050 2250 4050 2350
+Connection ~ 4050 2250
+Wire Wire Line
+	4200 2450 4050 2450
+Wire Wire Line
+	4050 2450 4050 2350
+Connection ~ 4050 2350
+$Comp
+L power:GND #PWR?
+U 1 1 5C725A2C
+P 4200 4950
+F 0 "#PWR?" H 4200 4700 50  0001 C CNN
+F 1 "GND" H 4205 4777 50  0000 C CNN
+F 2 "" H 4200 4950 50  0001 C CNN
+F 3 "" H 4200 4950 50  0001 C CNN
+	1    4200 4950
+	1    0    0    -1
+$EndComp
+Text GLabel 4200 4600 0    50   Input ~ 0
+TXD
+Text GLabel 4200 4700 0    50   Input ~ 0
+RXD
+Text GLabel 4200 3350 0    50   Input ~ 0
+EN
+Text GLabel 5900 2950 2    50   Input ~ 0
+IO0
 $EndSCHEMATC

Commit message: Im an Otter
Parts:
- removed R3: 100, symbol Device:R_Small
- C1, C2, C3: footprint (none) -> Capacitor_SMD:C_0402_1005Metric
- C4, C5, C6, C7: renamed from C?; footprint (none) -> Capacitor_SMD:C_0402_1005Metric
- Q1: footprint Package_TO_SOT_SMD:SOT-23 -> Package_TO_SOT_SMD:SOT-323_SC-70
- Q2: renamed from Q?; footprint Package_TO_SOT_SMD:SOT-23 -> Package_TO_SOT_SMD:SOT-323_SC-70
- Q3, Q4: renamed from Q?; footprint (none) -> Package_TO_SOT_SMD:SOT-323_SC-70
- R1, R2, R4: footprint (none) -> Resistor_SMD:R_0402_1005Metric
- R5: footprint (none) -> Resistor_SMD:R_0805_2012Metric
- R6, R7, R8: renamed from R?; footprint (none) -> Resistor_SMD:R_0402_1005Metric
- U3: renamed from U?; value CH340G -> CH340C
- U4: renamed from U?; footprint (none) -> badgelib:ST7789V; symbol anotterwatch-rescue:ST7789V-badgelib -> badgelib:ST7789V
- gave numbers to parts that had none: 2
Connections:
- net labels added: IPS_RST
Other:
- moved on the sheet: Q2, R6

Commit message: Im an Otter #2
Parts:
- added AE?: ANT, symbol Device:Antenna_Shield
- added C? (x2): 100n, Capacitor_SMD:C_0402_1005Metric, symbol Device:C_Small
- added C?: 10u, Capacitor_SMD:C_0402_1005Metric, symbol Device:C_Small
- added C? (x2): TBD, Capacitor_SMD:C_0402_1005Metric, symbol Device:C_Small
- added L?: TBD, symbol Device:L_Small
- added R?: 10k, Resistor_SMD:R_0402_1005Metric, symbol Device:R_Small
- Q1, Q2, Q3, Q4: footprint Package_TO_SOT_SMD:SOT-323_SC-70 -> Package_TO_SOT_SMD:SOT-23
- R5: value R_LED (150mA) -> 10
Connections:
- net EN: now also C?.1, R?.2
- net GND: now also AE?.2 (Shield), C?.2, C?.2, C?.2, C?.2, C?.2
- net VCC: now also U2.19 (VDD3P3_RTC), C?.1, C?.1, R?.1
- net at U2.2 (LNA_IN): now also C?.1, L?.1
- new net: AE?.1 (A), C?.1, L?.2
- no-connect marks 7 -> 9
Other:
- note added: "Todo: \nESP \nAFE (niklas) \nSensors (TBD)\nButtons\nBattery\n"
- note removed: "Todo: \nESP \nSerial-USB (with esd) \nDisplay\nAFE (niklas) \nSensors (TBD)\nButtons\nBattery\n"

Commit message: ADD: Analog Front-End
Parts:
- AE1: renamed from AE?; footprint (none) -> badgelib:Texas_SWRA117D_2.4GHz_Left
- C1, C2, C3, C4, C5, C6, C7: footprint Capacitor_SMD:C_0402_1005Metric -> Capacitor_SMD:C_0603_1608Metric
- C10, C11, C12, C8, C9: renamed from C?; footprint Capacitor_SMD:C_0402_1005Metric -> Capacitor_SMD:C_0603_1608Metric
- J1: symbol Connector:USB_C_Receptacle_USB2.0 -> anotterwatch-rescue:USB_C_Receptacle_USB2.0-Connector
- L1: renamed from L?; footprint (none) -> Inductor_SMD:L_0603_1608Metric
- R1, R2, R4, R6, R7, R8: footprint Resistor_SMD:R_0402_1005Metric -> Resistor_SMD:R_0603_1608Metric
- R3: renamed from R?; footprint Resistor_SMD:R_0402_1005Metric -> Resistor_SMD:R_0603_1608Metric
- R5: footprint Resistor_SMD:R_0805_2012Metric -> Resistor_SMD:R_0603_1608Metric
- U2: symbol ESP32-footprints-Shem-Lib:ESP32 -> anotterwatch-rescue:ESP32-ESP32-footprints-Shem-Lib
- U4: symbol badgelib:ST7789V -> anotterwatch-rescue:ST7789V-badgelib
Changed lines of the file:
@@
 $Descr A4 11693 8268
 encoding utf-8
-Sheet 1 1
+Sheet 1 2
 Title ""
 Date ""
@@
 Todo: \nESP \nAFE (niklas) \nSensors (TBD)\nButtons\nBattery\n
 $Comp
-L Connector:USB_C_Receptacle_USB2.0 J1
+L anotterwatch-rescue:USB_C_Receptacle_USB2.0-Connector J1
 U 1 1 5C6DC086
 P 1500 2950
@@
 F 0 "C1" H 1292 4096 50  0000 L CNN
 F 1 "100p" H 1292 4005 50  0000 L CNN
-F 2 "Capacitor_SMD:C_0402_1005Metric" H 1200 4050 50  0001 C CNN
+F 2 "Capacitor_SMD:C_0603_1608Metric" H 1200 4050 50  0001 C CNN
 F 3 "~" H 1200 4050 50  0001 C CNN
 	1    1200 4050
@@
 F 0 "R1" V 2350 2550 50  0000 C CNN
 F 1 "5k1" V 2245 2550 50  0000 C CNN
-F 2 "Resistor_SMD:R_0402_1005Metric" H 2350 2550 50  0001 C CNN
+F 2 "Resistor_SMD:R_0603_1608Metric" H 2350 2550 50  0001 C CNN
 F 3 "~" H 2350 2550 50  0001 C CNN
 	1    2350 2550
@@
 F 0 "R2" V 2350 2650 50  0000 C CNN
 F 1 "5k1" V 2450 2650 50  0000 C CNN
-F 2 "Resistor_SMD:R_0402_1005Metric" H 2350 2650 50  0001 C CNN
+F 2 "Resistor_SMD:R_0603_1608Metric" H 2350 2650 50  0001 C CNN
 F 3 "~" H 2350 2650 50  0001 C CNN
 	1    2350 2650
@@
 F 0 "C2" H 3142 6996 50  0000 L CNN
 F 1 "100n" H 3142 6905 50  0000 L CNN
-F 2 "Capacitor_SMD:C_0402_1005Metric" H 3050 6950 50  0001 C CNN
+F 2 "Capacitor_SMD:C_0603_1608Metric" H 3050 6950 50  0001 C CNN
 F 3 "~" H 3050 6950 50  0001 C CNN
 	1    3050 6950
@@
 F 0 "C3" H 3492 6996 50  0000 L CNN
 F 1 "100n" H 3492 6905 50  0000 L CNN
-F 2 "Capacitor_SMD:C_0402_1005Metric" H 3400 6950 50  0001 C CNN
+F 2 "Capacitor_SMD:C_0603_1608Metric" H 3400 6950 50  0001 C CNN
 F 3 "~" H 3400 6950 50  0001 C CNN
 	1    3400 6950
@@
 F 0 "R5" H 4959 6446 50  0000 L CNN
 F 1 "10" H 4959 6355 50  0000 L CNN
-F 2 "Resistor_SMD:R_0805_2012Metric" H 4900 6400 50  0001 C CNN
+F 2 "Resistor_SMD:R_0603_1608Metric" H 4900 6400 50  0001 C CNN
 F 3 "~" H 4900 6400 50  0001 C CNN
 	1    4900 6400
@@
 F 0 "R4" H 4559 7296 50  0000 L CNN
 F 1 "10k" H 4559 7205 50  0000 L CNN
-F 2 "Resistor_SMD:R_0402_1005Metric" H 4500 7250 50  0001 C CNN
+F 2 "Resistor_SMD:R_0603_1608Metric" H 4500 7250 50  0001 C CNN
 F 3 "~" H 4500 7250 50  0001 C CNN
 	1    4500 7250
@@
 $EndComp
 $Comp
-L badgelib:ST7789V U4
+L anotterwatch-rescue:ST7789V-badgelib U4
 U 1 1 5C7D4E59
 P 9750 5750
@@
 F 0 "R6" H 8359 5846 50  0000 L CNN
 F 1 "10k" H 8359 5755 50  0000 L CNN
-F 2 "Resistor_SMD:R_0402_1005Metric" H 8300 5800 50  0001 C CNN
+F 2 "Resistor_SMD:R_0603_1608Metric" H 8300 5800 50  0001 C CNN
 F 3 "~" H 8300 5800 50  0001 C CNN
 	1    8300 5800
@@
 F 0 "C6" H 10292 5796 50  0000 L CNN
 F 1 "100n" H 10292 5705 50  0000 L CNN
-F 2 "Capacitor_SMD:C_0402_1005Metric" H 10200 5750 50  0001 C CNN
+F 2 "Capacitor_SMD:C_0603_1608Metric" H 10200 5750 50  0001 C CNN
 F 3 "~" H 10200 5750 50  0001 C CNN
 	1    10200 5750
@@
 F 0 "C7" H 10692 5796 50  0000 L CNN
 F 1 "100n" H 10692 5705 50  0000 L CNN
-F 2 "Capacitor_SMD:C_0402_1005Metric" H 10600 5750 50  0001 C CNN
+F 2 "Capacitor_SMD:C_0603_1608Metric" H 10600 5750 50  0001 C CNN
 F 3 "~" H 10600 5750 50  0001 C CNN
 	1    10600 5750
@@
 F 0 "C5" H 8492 4296 50  0000 L CNN
 F 1 "100n" H 8492 4205 50  0000 L CNN
-F 2 "Capacitor_SMD:C_0402_1005Metric" H 8400 4250 50  0001 C CNN
+F 2 "Capacitor_SMD:C_0603_1608Metric" H 8400 4250 50  0001 C CNN
 F 3 "~" H 8400 4250 50  0001 C CNN
 	1    8400 4250
@@
 F 0 "C4" H 8142 4296 50  0000 L CNN
 F 1 "100n" H 8142 4205 50  0000 L CNN
-F 2 "Capacitor_SMD:C_0402_1005Metric" H 8050 4250 50  0001 C CNN
+F 2 "Capacitor_SMD:C_0603_1608Metric" H 8050 4250 50  0001 C CNN
 F 3 "~" H 8050 4250 50  0001 C CNN
 	1    8050 4250
@@
 F 0 "R7" V 10546 4000 50  0000 C CNN
 F 1 "10k" V 10455 4000 50  0000 C CNN
-F 2 "Resistor_SMD:R_0402_1005Metric" H 10350 4000 50  0001 C CNN
+F 2 "Resistor_SMD:R_0603_1608Metric" H 10350 4000 50  0001 C CNN
 F 3 "~" H 10350 4000 50  0001 C CNN
 	1    10350 4000
@@
 F 0 "R8" V 10154 4450 50  0000 C CNN
 F 1 "10k" V 10245 4450 50  0000 C CNN
-F 2 "Resistor_SMD:R_0402_1005Metric" H 10350 4450 50  0001 C CNN
+F 2 "Resistor_SMD:R_0603_1608Metric" H 10350 4450 50  0001 C CNN
 F 3 "~" H 10350 4450 50  0001 C CNN
 	1    10350 4450
@@
 EN
 $Comp
-L ESP32-footprints-Shem-Lib:ESP32 U2
+L anotterwatch-rescue:ESP32-ESP32-footprints-Shem-Lib U2
 U 1 1 5C71E383
 P 5050 3500
@@
 IPS_RST
 $Comp
-L Device:C_Small C?
+L Device:C_Small C10
 U 1 1 5C7354A0
 P 3600 2100
-F 0 "C?" H 3692 2146 50  0000 L CNN
+F 0 "C10" H 3692 2146 50  0000 L CNN
 F 1 "100n" H 3692 2055 50  0000 L CNN
-F 2 "Capacitor_SMD:C_0402_1005Metric" H 3600 2100 50  0001 C CNN
+F 2 "Capacitor_SMD:C_0603_1608Metric" H 3600 2100 50  0001 C CNN
 F 3 "~" H 3600 2100 50  0001 C CNN
 	1    3600 2100
@@
 $EndComp
 $Comp
-L power:GND #PWR?
+L power:GND #PWR05
 U 1 1 5C7354A7
 P 3600 2250
-F 0 "#PWR?" H 3600 2000 50  0001 C CNN
+F 0 "#PWR05" H 3600 2000 50  0001 C CNN
 F 1 "GND" H 3605 2077 50  0000 C CNN
 F 2 "" H 3600 2250 50  0001 C CNN
@@
 	3600 2250 3600 2200
 $Comp
-L Device:C_Small C?
+L Device:C_Small C8
 U 1 1 5C7368F7
 P 3250 2100
-F 0 "C?" H 3342 2146 50  0000 L CNN
+F 0 "C8" H 3342 2146 50  0000 L CNN
 F 1 "10u" H 3342 2055 50  0000 L CNN
-F 2 "Capacitor_SMD:C_0402_1005Metric" H 3250 2100 50  0001 C CNN
+F 2 "Capacitor_SMD:C_0603_1608Metric" H 3250 2100 50  0001 C CNN
 F 3 "~" H 3250 2100 50  0001 C CNN
 	1    3250 2100
@@
 $EndComp
 $Comp
-L power:GND #PWR?
+L power:GND #PWR02
 U 1 1 5C7368FE
 P 3250 2250
-F 0 "#PWR?" H 3250 2000 50  0001 C CNN
+F 0 "#PWR02" H 3250 2000 50  0001 C CNN
 F 1 "GND" H 3255 2077 50  0000 C CNN
 F 2 "" H 3250 2250 50  0001 C CNN
@@
 	3250 2250 3250 2200
 $Comp
-L power:VCC #PWR?
+L power:VCC #PWR01
 U 1 1 5C736906
 P 3250 1800
-F 0 "#PWR?" H 3250 1650 50  0001 C CNN
+F 0 "#PWR01" H 3250 1650 50  0001 C CNN
 F 1 "VCC" H 3267 1973 50  0000 C CNN
 F 2 "" H 3250 1800 50  0001 C CNN
@@
 NoConn ~ 4200 2600
 $Comp
-L Device:R_Small R?
+L Device:R_Small R3
 U 1 1 5C73EDA1
 P 3500 3200
-F 0 "R?" V 3696 3200 50  0000 C CNN
+F 0 "R3" V 3696 3200 50  0000 C CNN
 F 1 "10k" V 3605 3200 50  0000 C CNN
-F 2 "Resistor_SMD:R_0402_1005Metric" H 3500 3200 50  0001 C CNN
+F 2 "Resistor_SMD:R_0603_1608Metric" H 3500 3200 50  0001 C CNN
 F 3 "~" H 3500 3200 50  0001 C CNN
 	1    3500 3200
@@
 $EndComp
 $Comp
-L Device:C_Small C?
+L Device:C_Small C9
 U 1 1 5C7405C4
 P 3500 3500
-F 0 "C?" H 3592 3546 50  0000 L CNN
+F 0 "C9" H 3592 3546 50  0000 L CNN
 F 1 "100n" H 3592 3455 50  0000 L CNN
-F 2 "Capacitor_SMD:C_0402_1005Metric" H 3500 3500 50  0001 C CNN
+F 2 "Capacitor_SMD:C_0603_1608Metric" H 3500 3500 50  0001 C CNN
 F 3 "~" H 3500 3500 50  0001 C CNN
 	1    3500 3500
@@
 EN
 $Comp
-L power:GND #PWR?
+L power:GND #PWR04
 U 1 1 5C7438C6
 P 3500 3600
-F 0 "#PWR?" H 3500 3350 50  0001 C CNN
+F 0 "#PWR04" H 3500 3350 50  0001 C CNN
 F 1 "GND" H 3505 3427 50  0000 C CNN
 F 2 "" H 3500 3600 50  0001 C CNN
@@
 $EndComp
 $Comp
-L power:VCC #PWR?
+L power:VCC #PWR03
 U 1 1 5C7453B3
 P 3500 3100
-F 0 "#PWR?" H 3500 2950 50  0001 C CNN
+F 0 "#PWR03" H 3500 2950 50  0001 C CNN
 F 1 "VCC" H 3517 3273 50  0000 C CNN
 F 2 "" H 3500 3100 50  0001 C CNN
@@
 Connection ~ 3500 3350
 $Comp
-L power:VCC #PWR?
+L power:VCC #PWR06
 U 1 1 5C74C8E4
 P 6200 2250
-F 0 "#PWR?" H 6200 2100 50  0001 C CNN
+F 0 "#PWR06" H 6200 2100 50  0001 C CNN
 F 1 "VCC" H 6217 2423 50  0000 C CNN
 F 2 "" H 6200 2250 50  0001 C CNN
@@
 	5900 1950 6450 1950
 $Comp
-L Device:C_Small C?
+L Device:C_Small C11
 U 1 1 5C753AF6
 P 6450 2100
-F 0 "C?" H 6542 2146 50  0000 L CNN
+F 0 "C11" H 6542 2146 50  0000 L CNN
 F 1 "TBD" H 6542 2055 50  0000 L CNN
-F 2 "Capacitor_SMD:C_0402_1005Metric" H 6450 2100 50  0001 C CNN
+F 2 "Capacitor_SMD:C_0603_1608Metric" H 6450 2100 50  0001 C CNN
 F 3 "~" H 6450 2100 50  0001 C CNN
 	1    6450 2100
@@
 $EndComp
 $Comp
-L Device:C_Small C?
+L Device:C_Small C12
 U 1 1 5C755644
 P 6850 2100
-F 0 "C?" H 6942 2146 50  0000 L CNN
+F 0 "C12" H 6942 2146 50  0000 L CNN
 F 1 "TBD" H 6942 2055 50  0000 L CNN
-F 2 "Capacitor_SMD:C_0402_1005Metric" H 6850 2100 50  0001 C CNN
+F 2 "Capacitor_SMD:C_0603_1608Metric" H 6850 2100 50  0001 C CNN
 F 3 "~" H 6850 2100 50  0001 C CNN
 	1    6850 2100
@@
 $EndComp
 $Comp
-L power:GND #PWR?
+L power:GND #PWR07
 U 1 1 5C7571DC
 P 6450 2200
-F 0 "#PWR?" H 6450 1950 50  0001 C CNN
+F 0 "#PWR07" H 6450 1950 50  0001 C CNN
 F 1 "GND" H 6455 2027 50  0000 C CNN
 F 2 "" H 6450 2200 50  0001 C CNN
@@
 $EndComp
 $Comp
-L power:GND #PWR?
+L power:GND #PWR08
 U 1 1 5C75725E
 P 6850 2200
-F 0 "#PWR?" H 6850 1950 50  0001 C CNN
+F 0 "#PWR08" H 6850 1950 50  0001 C CNN
 F 1 "GND" H 6855 2027 50  0000 C CNN
 F 2 "" H 6850 2200 50  0001 C CNN
@@
 	6450 2000 6450 1950
 $Comp
-L Device:L_Small L?
+L Device:L_Small L1
 U 1 1 5C75B099
 P 6650 1950
-F 0 "L?" V 6835 1950 50  0000 C CNN
+F 0 "L1" V 6835 1950 50  0000 C CNN
 F 1 "TBD" V 6744 1950 50  0000 C CNN
-F 2 "" H 6650 1950 50  0001 C CNN
+F 2 "Inductor_SMD:L_0603_1608Metric" H 6650 1950 50  0001 C CNN
 F 3 "~" H 6650 1950 50  0001 C CNN
 	1    6650 1950
@@
 	6850 1950 7000 1950
 $Comp
-L Device:Antenna_Shield AE?
+L Device:Antenna_Shield AE1
 U 1 1 5C762CF6
 P 7000 1750
-F 0 "AE?" H 7141 1791 50  0000 L CNN
+F 0 "AE1" H 7141 1791 50  0000 L CNN
 F 1 "ANT" H 7141 1700 50  0000 L CNN
-F 2 "" H 7000 1850 50  0001 C CNN
+F 2 "badgelib:Texas_SWRA117D_2.4GHz_Left" H 7000 1850 50  0001 C CNN
 F 3 "~" H 7000 1850 50  0001 C CNN
 	1    7000 1750
@@
 $EndComp
 $Comp
-L power:GND #PWR?
+L power:GND #PWR09
 U 1 1 5C762D83
 P 7250 2000
-F 0 "#PWR?" H 7250 1750 50  0001 C CNN
+F 0 "#PWR09" H 7250 1750 50  0001 C CNN
 F 1 "GND" H 7255 1827 50  0000 C CNN
 F 2 "" H 7250 2000 50  0001 C CNN
@@
 IPS_RST
 NoConn ~ 2550 6950
+$Sheet
+S 8550 1200 2100 900
+U 5C72F19A
+F0 "Analog Front End" 50
+F1 "afe.sch" 50
+$EndSheet
 $EndSCHEMATC

Commit message: ADD: Jog switch
Parts:
- removed D2: SK6812, badgelib:sk6812_side, symbol LED:SK6812
- added S1: TMHU26, badgelib:TMHU26, symbol badgelib:TMHU26
- D3: footprint badgelib:RZX-S020CCW-0.4T -> LED_THT:LED_D5.0mm_Horizontal_O1.27mm_Z9.0mm
- J1: symbol anotterwatch-rescue:USB_C_Receptacle_USB2.0-Connector -> Connector:USB_C_Receptacle_USB2.0
- U2: symbol anotterwatch-rescue:ESP32-ESP32-footprints-Shem-Lib -> ESP32-footprints-Shem-Lib:ESP32
- U4: symbol anotterwatch-rescue:ST7789V-badgelib -> badgelib:ST7789V
Connections:
- wire segments 90 -> 87
- no-connect marks 9 -> 8
Changed lines of the file:
@@
 Todo: \nESP \nAFE (niklas) \nSensors (TBD)\nButtons\nBattery\n
 $Comp
-L anotterwatch-rescue:USB_C_Receptacle_USB2.0-Connector J1
+L Connector:USB_C_Receptacle_USB2.0 J1
 U 1 1 5C6DC086
 P 1500 2950
@@
 Wire Wire Line
 	1500 5900 1500 5800
-$Comp
-L LED:SK6812 D2
-U 1 1 5C6E3E9C
-P 2250 6950
-F 0 "D2" H 2591 6996 50  0000 L CNN
-F 1 "SK6812" H 2591 6905 50  0000 L CNN
-F 2 "badgelib:sk6812_side" H 2300 6650 50  0001 L TNN
-F 3 "https://de.aliexpress.com/item/10-3000-st-cke-SK6812-4020-Seite-Emmitting-RGB-LED-mit-eingebauten-SK6812-IC-SMD-4020/32877531241.html" H 2350 6575 50  0001 L TNN
-F 4 "SK6812 4020" H 2250 6950 50  0001 C CNN "Type"
-	1    2250 6950
-	1    0    0    -1
-$EndComp
-Wire Wire Line
-	1950 6950 1550 6950
 Wire Wire Line
 	1250 6600 1250 6650
-Wire Wire Line
-	2250 6650 2250 6600
-$Comp
-L power:GND #PWR0109
-U 1 1 5C6E4795
-P 2250 7300
-F 0 "#PWR0109" H 2250 7050 50  0001 C CNN
-F 1 "GND" H 2255 7127 50  0000 C CNN
-F 2 "" H 2250 7300 50  0001 C CNN
-F 3 "" H 2250 7300 50  0001 C CNN
-	1    2250 7300
-	1    0    0    -1
-$EndComp
-Wire Wire Line
-	2250 7300 2250 7250
 $Comp
 L power:GND #PWR0110
@@
 F 0 "D3" V 4938 6583 50  0000 R CNN
 F 1 "LED" V 4847 6583 50  0000 R CNN
-F 2 "badgelib:RZX-S020CCW-0.4T" H 4900 6700 50  0001 C CNN
+F 2 "LED_THT:LED_D5.0mm_Horizontal_O1.27mm_Z9.0mm" H 4900 6700 50  0001 C CNN
 F 3 "https://de.aliexpress.com/item/2000-st-cke-Rolle-Ultra-slim-0-4mm-seite-view-LED-020-SMD-geeignet-f-r/32920375451.html" H 4900 6700 50  0001 C CNN
 F 4 "RZX-S020CCW-0.4T" V 4900 6700 50  0001 C CNN "Type"
@@
 $EndComp
 $Comp
-L anotterwatch-rescue:ST7789V-badgelib U4
+L badgelib:ST7789V U4
 U 1 1 5C7D4E59
 P 9750 5750
@@
 F 3 "" H 3050 6800 50  0001 C CNN
 	1    3050 6800
-	1    0    0    -1
-$EndComp
-$Comp
-L power:VCC #PWR0108
-U 1 1 5C7D6EEF
-P 2250 6600
-F 0 "#PWR0108" H 2250 6450 50  0001 C CNN
-F 1 "VCC" H 2267 6773 50  0000 C CNN
-F 2 "" H 2250 6600 50  0001 C CNN
-F 3 "" H 2250 6600 50  0001 C CNN
-	1    2250 6600
 	1    0    0    -1
 $EndComp
@@
 Text GLabel 10950 3800 1    50   Input ~ 0
 EN
-$Comp
-L anotterwatch-rescue:ESP32-ESP32-footprints-Shem-Lib U2
-U 1 1 5C71E383
-P 5050 3500
-F 0 "U2" H 5050 5337 60  0000 C CNN
-F 1 "ESP32" H 5050 5231 60  0000 C CNN
-F 2 "ESP32-footprints-Lib:ESP32" H 5050 1875 60  0001 C CNN
-F 3 "https://www.espressif.com/sites/default/files/documentation/esp32-pico-d4_datasheet_en.pdf" H 5500 4400 60  0001 C CNN
-F 4 "https://github.com/adamjvr/ESP32-kiCAD-Footprints" H 5050 3500 50  0001 C CNN "Lib"
-	1    5050 3500
-	1    0    0    -1
-$EndComp
 Wire Wire Line
 	4200 1950 4050 1950
@@
 Text GLabel 3500 4800 0    50   Input ~ 0
 IPS_RST
-NoConn ~ 2550 6950
 $Sheet
 S 8550 1200 2100 900
@@
 F1 "afe.sch" 50
 $EndSheet
+$Comp
+L badgelib:TMHU26 S1
+U 1 1 5C731DCE
+P 7850 2700
+F 0 "S1" H 7850 3025 50  0000 C CNN
+F 1 "TMHU26" H 7850 2934 50  0000 C CNN
+F 2 "badgelib:TMHU26" H 7850 2900 50  0001 C CNN
+F 3 "" H 7850 2900 50  0001 C CNN
+	1    7850 2700
+	1    0    0    -1
+$EndComp
+$Comp
+L ESP32-footprints-Shem-Lib:ESP32 U2
+U 1 1 5C71E383
+P 5050 3500
+F 0 "U2" H 5050 5337 60  0000 C CNN
+F 1 "ESP32" H 5050 5231 60  0000 C CNN
+F 2 "ESP32-footprints-Lib:ESP32" H 5050 1875 60  0001 C CNN
+F 3 "https://www.espressif.com/sites/default/files/documentation/esp32-pico-d4_datasheet_en.pdf" H 5500 4400 60  0001 C CNN
+F 4 "https://github.com/adamjvr/ESP32-kiCAD-Footprints" H 5050 3500 50  0001 C CNN "Lib"
+	1    5050 3500
+	1    0    0    -1
+$EndComp
 $EndSCHEMATC
