File: Power.sch (KiCad schematic (older format))
At the start: 10 parts, among them J1 USB_C_Receptacle_USB2.0

Commit message: Schematic cleanup
Parts:
- removed L?: 2.2u, symbol Device:L
- added C2, C27: 100n, Capacitor_SMD:C_0603_1608Metric, symbol Device:C_Small
- added J4: Conn_01x02_Female, symbol Connector:Conn_01x02_Female
- added L2: 2.2u, symbol Device:L
- added R36: 47k, Resistor_SMD:R_0603_1608Metric, symbol Device:R_Small
- added R43: 2k5, Resistor_SMD:R_0603_1608Metric, symbol Device:R_Small
- added U1: TP4056, Package_SO:Diodes_PSOP-8, symbol badgelib:TP4056
- added U14: TPS63001DRCR, Package_SON:Texas_S-PVSON-N10, symbol TPS63001DRCR:TPS63001DRCR
- gave numbers to parts that had none: 5
Connections:
- net labels added: +3.3V, +BATT, CHRG, TPS_FB
- wire segments 44 -> 51
Other:
- moved on the sheet: C26, C28, C29, C3, R47

Commit message: added datasheets and descriptions
Parts:
- J4: value Conn_01x02_Female -> Bat
Other:
- note added: "2k -> 580mA\n3k -> 400mA\n4k -> 300mA\n5k1 -> 240mA"
- note added: "Battery Charging"
- note added: "JST 2.0mm 2pin, need to find out type and pinout"
- note added: "TODO: Ideal diode!"
- note added: "VBAT to 3.3V Buck-Boost"
Changed lines of the file:
@@
 F 1 "TPS63001DRCR" H 6300 3879 50  0000 C CNN
 F 2 "Package_SON:Texas_S-PVSON-N10" H 6300 3100 50  0001 L BNN
-F 3 "Converter DC-DC Single Non-Inverting/Inverting/Step Up/Step Down 1.8V to 5.5V 10-Pin VSON EP T/R" H 6300 3100 50  0001 L BNN
+F 3 "http://www.ti.com/lit/ds/symlink/tps63001.pdf" H 6300 3100 50  0001 L BNN
 F 4 "None" H 6300 3100 50  0001 L BNN "Field4"
 F 5 "Unavailable" H 6300 3100 50  0001 L BNN "Field5"
@@
 F 1 "TP4056" H 4050 6024 50  0000 C CNN
 F 2 "Package_SO:Diodes_PSOP-8" H 4050 5700 50  0001 C CNN
-F 3 "" H 4050 5700 50  0001 C CNN
+F 3 "https://dlnmh9ip6v2uc.cloudfront.net/datasheets/Prototyping/TP4056.pdf" H 4050 5700 50  0001 C CNN
 	1    4050 5700
 	1    0    0    -1
@@
 P 6700 5350
 F 0 "J4" H 6594 5025 50  0000 C CNN
-F 1 "Conn_01x02_Female" H 6594 5116 50  0000 C CNN
+F 1 "Bat" H 6594 5116 50  0000 C CNN
 F 2 "" H 6700 5350 50  0001 C CNN
 F 3 "~" H 6700 5350 50  0001 C CNN
@@
 	0    1    1    0
 $EndComp
+Text Notes 5850 4950 0    50   ~ 0
+JST 2.0mm 2pin, need to find out type and pinout
+Text Notes 2800 4650 0    197  ~ 0
+TODO: Ideal diode!
+Text Notes 4900 2050 0    79   ~ 0
+VBAT to 3.3V Buck-Boost
+Text Notes 3550 5150 0    79   ~ 0
+Battery Charging
+Text Notes 4750 6350 0    50   ~ 0
+2k -> 580mA\n3k -> 400mA\n4k -> 300mA\n5k1 -> 240mA
 $EndSCHEMATC
