File: power.sch (KiCad schematic (older format))
At the start: 17 parts, among them J1 USB_C_Receptacle_USB2.0, J4 Bat, U1 TP4056, U14 TPS63001DRCR

Commit message: add anotation
Parts:
- J4: footprint (none) -> Connector_JST:JST_PH_B2B-PH-SM4-TB_1x02-1MP_P2.00mm_Vertical
- L2: footprint (none) -> Inductor_SMD:L_Taiyo-Yuden_MD-3030
Changed lines of the file:
@@
 F 0 "L2" V 5400 3300 50  0000 C CNN
 F 1 "2.2u" V 5250 3300 50  0000 C CNN
-F 2 "" H 5300 3300 50  0001 C CNN
+F 2 "Inductor_SMD:L_Taiyo-Yuden_MD-3030" H 5300 3300 50  0001 C CNN
 F 3 "~" H 5300 3300 50  0001 C CNN
 	1    5300 3300
@@
 F 0 "J4" H 6594 5025 50  0000 C CNN
 F 1 "Bat" H 6594 5116 50  0000 C CNN
-F 2 "" H 6700 5350 50  0001 C CNN
+F 2 "Connector_JST:JST_PH_B2B-PH-SM4-TB_1x02-1MP_P2.00mm_Vertical" H 6700 5350 50  0001 C CNN
 F 3 "~" H 6700 5350 50  0001 C CNN
 	1    6700 5350

Commit message: UPD: finalized schematic, started layout
Parts:
- removed C2: 100n, Capacitor_SMD:C_0603_1608Metric, symbol Device:C_Small
- removed J4: Bat, Connector_JST:JST_PH_B2B-PH-SM4-TB_1x02-1MP_P2.00mm_Vertical, symbol Connector:Conn_01x02_Female
- removed R43: 2k5, Resistor_SMD:R_0603_1608Metric, symbol Device:R_Small
- added BT1: 603020, Connector_JST:JST_GH_BM02B-GHS-TBT_1x02-1MP_P1.25mm_Vertical, symbol Device:Battery_Cell
- added C25: 10u, Capacitor_SMD:C_0603_1608Metric, symbol Device:C_Small
- added D7: D_Small, Diode_SMD:D_SMA, symbol Device:D_Small
- added Q10: Q_PMOS_GDS, Package_TO_SOT_SMD:SOT-23, symbol Device:Q_PMOS_GDS
- added R44, R45: 5k1, Resistor_SMD:R_0603_1608Metric, symbol Device:R_Small
- added R46: 47k, Resistor_SMD:R_0603_1608Metric, symbol Device:R_Small
- added SW1: SW_SPST, Button_Switch_SMD:SW_SPDT_PCM12, symbol Switch:SW_SPST
- C26: renamed from C27; value 100n -> 10u
- R43: renamed from R36; value 47k -> 390k
- U14: symbol TPS63001DRCR:TPS63001DRCR -> anotterwatch-rescue:TPS63001DRCR-TPS63001DRCR
- renumbered C1 to C24, C3 to C27, C26 to C28, C28 to C29, C29 to C30, J1 to J4, R1 to R41, R2 to R42, U1 to U13
Connections:
- net labels removed: TPS_FB
- wire segments 51 -> 66
Other:
- note removed: "2k -> 580mA\n3k -> 400mA\n4k -> 300mA\n5k1 -> 240mA"
- note removed: "JST 2.0mm 2pin, need to find out type and pinout"
- note removed: "TODO: Ideal diode!"
- moved on the sheet: C24, C26, C27, C28, C29, C30, J4, L2, R41, R42, R43, R47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

Commit message: ADD: constant current source for high power LED
Parts:
- renumbered D7 to D6, R41 to R45, R42 to R46, R43 to R47, R44 to R48, R45 to R49, R46 to R50, R47 to R51
Changed lines of the file:
@@
 encoding utf-8
 Sheet 3 3
-Title ""
+Title "anOtter Watch"
 Date ""
-Rev ""
-Comp ""
-Comment1 ""
+Rev "V1.0"
+Comp "A badge.team Project"
+Comment1 "HW design by Jan Henrik and Niklas"
 Comment2 ""
 Comment3 ""
@@
 $EndComp
 $Comp
-L Device:R_Small R41
+L Device:R_Small R45
 U 1 1 5C753E35
 P 2400 2950
-F 0 "R41" V 2400 2950 50  0000 C CNN
+F 0 "R45" V 2400 2950 50  0000 C CNN
 F 1 "5k1" V 2295 2950 50  0000 C CNN
 F 2 "Resistor_SMD:R_0603_1608Metric" H 2400 2950 50  0001 C CNN
@@
 $EndComp
 $Comp
-L Device:R_Small R42
+L Device:R_Small R46
 U 1 1 5C753E3C
 P 2400 3050
-F 0 "R42" V 2400 3050 50  0000 C CNN
+F 0 "R46" V 2400 3050 50  0000 C CNN
 F 1 "5k1" V 2500 3050 50  0000 C CNN
 F 2 "Resistor_SMD:R_0603_1608Metric" H 2400 3050 50  0001 C CNN
@@
 	2700 2950 2500 2950
 $Comp
-L power:GND #PWR094
+L power:GND #PWR095
 U 1 1 5C753E4A
 P 2700 3050
-F 0 "#PWR094" H 2700 2800 50  0001 C CNN
+F 0 "#PWR095" H 2700 2800 50  0001 C CNN
 F 1 "GND" H 2705 2877 50  0000 C CNN
 F 2 "" H 2700 3050 50  0001 C CNN
@@
 P 1550 4300
 AR Path="/5C7642A4" Ref="#PWR?"  Part="1"
-AR Path="/5C753B69/5C7642A4" Ref="#PWR093"  Part="1"
-F 0 "#PWR093" H 1550 4050 50  0001 C CNN
+AR Path="/5C753B69/5C7642A4" Ref="#PWR094"  Part="1"
+F 0 "#PWR094" H 1550 4050 50  0001 C CNN
 F 1 "GND" H 1555 4127 50  0000 C CNN
 F 2 "" H 1550 4300 50  0001 C CNN
@@
 $EndComp
 $Comp
-L power:GND #PWR0109
+L power:GND #PWR0110
 U 1 1 5C776CB5
 P 8300 4100
-F 0 "#PWR0109" H 8300 3850 50  0001 C CNN
+F 0 "#PWR0110" H 8300 3850 50  0001 C CNN
 F 1 "GND" H 8305 3927 50  0000 C CNN
 F 2 "" H 8300 4100 50  0001 C CNN
@@
 $EndComp
 $Comp
-L Device:R_Small R47
+L Device:R_Small R51
 U 1 1 5C777E0D
 P 7500 2900
-F 0 "R47" V 7600 2900 50  0000 C CNN
+F 0 "R51" V 7600 2900 50  0000 C CNN
 F 1 "100" V 7395 2900 50  0000 C CNN
 F 2 "Resistor_SMD:R_0603_1608Metric" H 7500 2900 50  0001 C CNN
@@
 Connection ~ 7500 2750
 $Comp
-L power:GND #PWR0107
+L power:GND #PWR0108
 U 1 1 5C779A9F
 P 7500 3350
-F 0 "#PWR0107" H 7500 3100 50  0001 C CNN
+F 0 "#PWR0108" H 7500 3100 50  0001 C CNN
 F 1 "GND" H 7505 3177 50  0000 C CNN
 F 2 "" H 7500 3350 50  0001 C CNN
@@
 	9950 2750 10300 2750
 $Comp
-L power:GND #PWR0106
+L power:GND #PWR0107
 U 1 1 5C77E653
 P 7050 2950
-F 0 "#PWR0106" H 7050 2700 50  0001 C CNN
+F 0 "#PWR0107" H 7050 2700 50  0001 C CNN
 F 1 "GND" H 7055 2777 50  0000 C CNN
 F 2 "" H 7050 2950 50  0001 C CNN
@@
 $EndComp
 $Comp
-L power:GND #PWR0110
+L power:GND #PWR0111
 U 1 1 5C77ED9A
 P 9950 2950
-F 0 "#PWR0110" H 9950 2700 50  0001 C CNN
+F 0 "#PWR0111" H 9950 2700 50  0001 C CNN
 F 1 "GND" H 9955 2777 50  0000 C CNN
 F 2 "" H 9950 2950 50  0001 C CNN
@@
 $EndComp
 $Comp
-L power:GND #PWR0112
+L power:GND #PWR0113
 U 1 1 5C77F4E1
 P 10300 2950
-F 0 "#PWR0112" H 10300 2700 50  0001 C CNN
+F 0 "#PWR0113" H 10300 2700 50  0001 C CNN
 F 1 "GND" H 10305 2777 50  0000 C CNN
 F 2 "" H 10300 2950 50  0001 C CNN
@@
 P 10300 2750
 AR Path="/5C79E309" Ref="#PWR?"  Part="1"
-AR Path="/5C753B69/5C79E309" Ref="#PWR0111"  Part="1"
-F 0 "#PWR0111" H 10300 2600 50  0001 C CNN
+AR Path="/5C753B69/5C79E309" Ref="#PWR0112"  Part="1"
+F 0 "#PWR0112" H 10300 2600 50  0001 C CNN
 F 1 "+3.3V" H 10315 2923 50  0000 C CNN
 F 2 "" H 10300 2750 50  0001 C CNN
@@
 P 4400 3050
 AR Path="/5C7A88B5" Ref="#PWR?"  Part="1"
-AR Path="/5C753B69/5C7A88B5" Ref="#PWR098"  Part="1"
-F 0 "#PWR098" H 4400 2800 50  0001 C CNN
+AR Path="/5C753B69/5C7A88B5" Ref="#PWR099"  Part="1"
+F 0 "#PWR099" H 4400 2800 50  0001 C CNN
 F 1 "GND" H 4405 2877 50  0000 C CNN
 F 2 "" H 4400 3050 50  0001 C CNN
@@
 P 4600 3150
 AR Path="/5C7A88E0" Ref="#PWR?"  Part="1"
-AR Path="/5C753B69/5C7A88E0" Ref="#PWR0100"  Part="1"
-F 0 "#PWR0100" H 4600 2900 50  0001 C CNN
+AR Path="/5C753B69/5C7A88E0" Ref="#PWR0101"  Part="1"
+F 0 "#PWR0101" H 4600 2900 50  0001 C CNN
 F 1 "GND" H 4605 2977 50  0000 C CNN
 F 2 "" H 4600 3150 50  0001 C CNN
@@
 P 5100 3050
 AR Path="/5C7A88EE" Ref="#PWR?"  Part="1"
-AR Path="/5C753B69/5C7A88EE" Ref="#PWR0102"  Part="1"
-F 0 "#PWR0102" H 5100 2800 50  0001 C CNN
+AR Path="/5C753B69/5C7A88EE" Ref="#PWR0103"  Part="1"
+F 0 "#PWR0103" H 5100 2800 50  0001 C CNN
 F 1 "GND" H 5105 2877 50  0000 C CNN
 F 2 "" H 5100 3050 50  0001 C CNN
@@
 P 4500 2850
 AR Path="/5C7A88F6" Ref="#PWR?"  Part="1"
-AR Path="/5C753B69/5C7A88F6" Ref="#PWR099"  Part="1"
-F 0 "#PWR099" H 4500 2600 50  0001 C CNN
+AR Path="/5C753B69/5C7A88F6" Ref="#PWR0100"  Part="1"
+F 0 "#PWR0100" H 4500 2600 50  0001 C CNN
 F 1 "GND" V 4500 2650 50  0000 C CNN
 F 2 "" H 4500 2850 50  0001 C CNN
@@
 P 2900 3650
 AR Path="/5C7A8902" Ref="R?"  Part="1"
-AR Path="/5C753B69/5C7A8902" Ref="R43"  Part="1"
-F 0 "R43" V 3096 3650 50  0000 C CNN
+AR Path="/5C753B69/5C7A8902" Ref="R47"  Part="1"
+F 0 "R47" V 3096 3650 50  0000 C CNN
 F 1 "390k" V 3005 3650 50  0000 C CNN
 F 2 "Resistor_SMD:R_0603_1608Metric" H 2900 3650 50  0001 C CNN
@@
 P 2900 3550
 AR Path="/5C7A8909" Ref="#PWR?"  Part="1"
-AR Path="/5C753B69/5C7A8909" Ref="#PWR096"  Part="1"
-F 0 "#PWR096" H 2900 3400 50  0001 C CNN
+AR Path="/5C753B69/5C7A8909" Ref="#PWR097"  Part="1"
+F 0 "#PWR097" H 2900 3400 50  0001 C CNN
 F 1 "+3.3V" H 2915 3723 50  0000 C CNN
 F 2 "" H 2900 3550 50  0001 C CNN
@@
 $EndComp
 $Comp
-L power:GND #PWR0103
+L power:GND #PWR0104
 U 1 1 5CBC44E0
 P 5500 3050
-F 0 "#PWR0103" H 5500 2800 50  0001 C CNN
+F 0 "#PWR0104" H 5500 2800 50  0001 C CNN
 F 1 "GND" H 5505 2877 50  0000 C CNN
 F 2 "" H 5500 3050 50  0001 C CNN
@@
 P 6400 3200
 AR Path="/5CBCC521" Ref="R?"  Part="1"
-AR Path="/5C753B69/5CBCC521" Ref="R46"  Part="1"
-F 0 "R46" H 6550 3300 50  0000 C CNN
+AR Path="/5C753B69/5CBCC521" Ref="R50"  Part="1"
+F 0 "R50" H 6550 3300 50  0000 C CNN
 F 1 "47k" H 6550 3200 50  0000 C CNN
 F 2 "Resistor_SMD:R_0603_1608Metric" H 6400 3200 50  0001 C CNN
@@
 $EndComp
 $Comp
-L power:GND #PWR0104
+L power:GND #PWR0105
 U 1 1 5CBCC5D2
 P 6400 3300
-F 0 "#PWR0104" H 6400 3050 50  0001 C CNN
+F 0 "#PWR0105" H 6400 3050 50  0001 C CNN
 F 1 "GND" H 6550 3250 50  0000 C CNN
 F 2 "" H 6400 3300 50  0001 C CNN
@@
 $EndComp
 $Comp
-L power:VBUS #PWR097
+L power:VBUS #PWR098
 U 1 1 5CBD124C
 P 3500 2750
-F 0 "#PWR097" H 3500 2600 50  0001 C CNN
+F 0 "#PWR098" H 3500 2600 50  0001 C CNN
 F 1 "VBUS" H 3515 2923 50  0000 C CNN
 F 2 "" H 3500 2750 50  0001 C CNN
@@
 Connection ~ 6400 3050
 $Comp
-L Device:D_Small D7
+L Device:D_Small D6
 U 1 1 5CBD4020
 P 6400 3550
-F 0 "D7" H 6400 3450 50  0000 C CNN
+F 0 "D6" H 6400 3450 50  0000 C CNN
 F 1 "D_Small" H 6400 3650 50  0000 C CNN
 F 2 "Diode_SMD:D_SMA" V 6400 3550 50  0001 C CNN
@@
 P 2900 3050
 AR Path="/5CBDD97E" Ref="#PWR?"  Part="1"
-AR Path="/5C753B69/5CBDD97E" Ref="#PWR095"  Part="1"
-F 0 "#PWR095" H 2900 2800 50  0001 C CNN
+AR Path="/5C753B69/5CBDD97E" Ref="#PWR096"  Part="1"
+F 0 "#PWR096" H 2900 2800 50  0001 C CNN
 F 1 "GND" H 2905 2877 50  0000 C CNN
 F 2 "" H 2900 3050 50  0001 C CNN
@@
 P 7050 2750
 AR Path="/5CBE39C6" Ref="#PWR?"  Part="1"
-AR Path="/5C753B69/5CBE39C6" Ref="#PWR0105"  Part="1"
-F 0 "#PWR0105" H 7050 2600 50  0001 C CNN
+AR Path="/5C753B69/5CBE39C6" Ref="#PWR0106"  Part="1"
+F 0 "#PWR0106" H 7050 2600 50  0001 C CNN
 F 1 "+BATT" H 6950 2900 50  0000 L CNN
 F 2 "" H 7050 2750 50  0001 C CNN
@@
 P 8150 3150
 AR Path="/5CBF3C84" Ref="#PWR?"  Part="1"
-AR Path="/5C753B69/5CBF3C84" Ref="#PWR0108"  Part="1"
-F 0 "#PWR0108" H 8150 3000 50  0001 C CNN
+AR Path="/5C753B69/5CBF3C84" Ref="#PWR0109"  Part="1"
+F 0 "#PWR0109" H 8150 3000 50  0001 C CNN
 F 1 "+3.3V" V 8150 3400 50  0000 C CNN
 F 2 "" H 8150 3150 50  0001 C CNN
@@
 $EndComp
 $Comp
-L Device:R_Small R44
+L Device:R_Small R48
 U 1 1 5CC15309
 P 4600 3050
-F 0 "R44" V 4600 3050 50  0000 C CNN
+F 0 "R48" V 4600 3050 50  0000 C CNN
 F 1 "5k1" V 4700 3050 50  0000 C CNN
 F 2 "Resistor_SMD:R_0603_1608Metric" H 4600 3050 50  0001 C CNN
@@
 $EndComp
 $Comp
-L Device:R_Small R45
+L Device:R_Small R49
 U 1 1 5CC1540B
 P 4800 3050
-F 0 "R45" V 4800 3050 50  0000 C CNN
+F 0 "R49" V 4800 3050 50  0000 C CNN
 F 1 "5k1" V 4900 3050 50  0000 C CNN
 F 2 "Resistor_SMD:R_0603_1608Metric" H 4800 3050 50  0001 C CNN
@@
 P 4800 3150
 AR Path="/5CC16ABF" Ref="#PWR?"  Part="1"
-AR Path="/5C753B69/5CC16ABF" Ref="#PWR0101"  Part="1"
-F 0 "#PWR0101" H 4800 2900 50  0001 C CNN
+AR Path="/5C753B69/5CC16ABF" Ref="#PWR0102"  Part="1"
+F 0 "#PWR0102" H 4800 2900 50  0001 C CNN
 F 1 "GND" H 4805 2977 50  0000 C CNN
 F 2 "" H 4800 3150 50  0001 C CNN

Commit message: ADD:started to place footprints
Parts:
- removed Q10: Q_PMOS_GDS, Package_TO_SOT_SMD:SOT-23, symbol Device:Q_PMOS_GDS
- added Q10: Q_PMOS_GSD, symbol Device:Q_PMOS_GSD
- C24, C28, C29: footprint Capacitor_SMD:C_0603_1608Metric -> Capacitor_SMD:C_0402_1005Metric
- D6: footprint Diode_SMD:D_SMA -> Diode_SMD:D_SOD-123F
- R45, R46, R47, R48, R49, R50, R51: footprint Resistor_SMD:R_0603_1608Metric -> Resistor_SMD:R_0402_1005Metric
Connections:
- net +BATT: now also Q10.3 (D)
- net VBUS: now also Q10.1 (G)
- net at SW1.2 (B): now also Q10.2 (S)
Changed lines of the file:
@@
 F 0 "R45" V 2400 2950 50  0000 C CNN
 F 1 "5k1" V 2295 2950 50  0000 C CNN
-F 2 "Resistor_SMD:R_0603_1608Metric" H 2400 2950 50  0001 C CNN
+F 2 "Resistor_SMD:R_0402_1005Metric" H 2400 2950 50  0001 C CNN
 F 3 "~" H 2400 2950 50  0001 C CNN
 	1    2400 2950
@@
 F 0 "R46" V 2400 3050 50  0000 C CNN
 F 1 "5k1" V 2500 3050 50  0000 C CNN
-F 2 "Resistor_SMD:R_0603_1608Metric" H 2400 3050 50  0001 C CNN
+F 2 "Resistor_SMD:R_0402_1005Metric" H 2400 3050 50  0001 C CNN
 F 3 "~" H 2400 3050 50  0001 C CNN
 	1    2400 3050
@@
 F 0 "C24" V 1550 3950 50  0000 L CNN
 F 1 "100p" V 1550 4100 50  0000 L CNN
-F 2 "Capacitor_SMD:C_0603_1608Metric" H 1400 4250 50  0001 C CNN
+F 2 "Capacitor_SMD:C_0402_1005Metric" H 1400 4250 50  0001 C CNN
 F 3 "~" H 1400 4250 50  0001 C CNN
 	1    1400 4250
@@
 F 0 "C28" H 7592 3296 50  0000 L CNN
 F 1 "100n" H 7592 3205 50  0000 L CNN
-F 2 "Capacitor_SMD:C_0603_1608Metric" H 7500 3250 50  0001 C CNN
+F 2 "Capacitor_SMD:C_0402_1005Metric" H 7500 3250 50  0001 C CNN
 F 3 "~" H 7500 3250 50  0001 C CNN
 	1    7500 3250
@@
 F 0 "R51" V 7600 2900 50  0000 C CNN
 F 1 "100" V 7395 2900 50  0000 C CNN
-F 2 "Resistor_SMD:R_0603_1608Metric" H 7500 2900 50  0001 C CNN
+F 2 "Resistor_SMD:R_0402_1005Metric" H 7500 2900 50  0001 C CNN
 F 3 "~" H 7500 2900 50  0001 C CNN
 	1    7500 2900
@@
 F 0 "C29" H 10042 2896 50  0000 L CNN
 F 1 "100n" H 10042 2805 50  0000 L CNN
-F 2 "Capacitor_SMD:C_0603_1608Metric" H 9950 2850 50  0001 C CNN
+F 2 "Capacitor_SMD:C_0402_1005Metric" H 9950 2850 50  0001 C CNN
 F 3 "~" H 9950 2850 50  0001 C CNN
 	1    9950 2850
@@
 F 0 "R47" V 3096 3650 50  0000 C CNN
 F 1 "390k" V 3005 3650 50  0000 C CNN
-F 2 "Resistor_SMD:R_0603_1608Metric" H 2900 3650 50  0001 C CNN
+F 2 "Resistor_SMD:R_0402_1005Metric" H 2900 3650 50  0001 C CNN
 F 3 "~" H 2900 3650 50  0001 C CNN
 	1    2900 3650
@@
 $EndComp
 Connection ~ 5100 2750
-$Comp
-L Device:Q_PMOS_GDS Q10
-U 1 1 5CBC71E1
-P 6400 2850
-F 0 "Q10" V 6750 3100 50  0000 C CNN
-F 1 "Q_PMOS_GDS" V 6650 2900 50  0000 C CNN
-F 2 "Package_TO_SOT_SMD:SOT-23" H 6600 2950 50  0001 C CNN
-F 3 "~" H 6400 2850 50  0001 C CNN
-	1    6400 2850
-	0    -1   -1   0
-$EndComp
 Wire Wire Line
 	5100 2800 5100 2750
@@
 F 0 "R50" H 6550 3300 50  0000 C CNN
 F 1 "47k" H 6550 3200 50  0000 C CNN
-F 2 "Resistor_SMD:R_0603_1608Metric" H 6400 3200 50  0001 C CNN
+F 2 "Resistor_SMD:R_0402_1005Metric" H 6400 3200 50  0001 C CNN
 F 3 "~" H 6400 3200 50  0001 C CNN
 	1    6400 3200
@@
 Wire Wire Line
 	6400 3100 6400 3050
-Connection ~ 6400 3050
 $Comp
 L Device:D_Small D6
@@
 F 0 "D6" H 6400 3450 50  0000 C CNN
 F 1 "D_Small" H 6400 3650 50  0000 C CNN
-F 2 "Diode_SMD:D_SMA" V 6400 3550 50  0001 C CNN
+F 2 "Diode_SMD:D_SOD-123F" V 6400 3550 50  0001 C CNN
 F 3 "~" V 6400 3550 50  0001 C CNN
 	1    6400 3550
@@
 F 0 "R48" V 4600 3050 50  0000 C CNN
 F 1 "5k1" V 4700 3050 50  0000 C CNN
-F 2 "Resistor_SMD:R_0603_1608Metric" H 4600 3050 50  0001 C CNN
+F 2 "Resistor_SMD:R_0402_1005Metric" H 4600 3050 50  0001 C CNN
 F 3 "~" H 4600 3050 50  0001 C CNN
 	1    4600 3050
@@
 F 0 "R49" V 4800 3050 50  0000 C CNN
 F 1 "5k1" V 4900 3050 50  0000 C CNN
-F 2 "Resistor_SMD:R_0603_1608Metric" H 4800 3050 50  0001 C CNN
+F 2 "Resistor_SMD:R_0402_1005Metric" H 4800 3050 50  0001 C CNN
 F 3 "~" H 4800 3050 50  0001 C CNN
 	1    4800 3050
@@
 	5650 2750 5500 2750
 Connection ~ 5500 2750
+$Comp
+L Device:Q_PMOS_GSD Q?
+U 1 1 5CE12F3D
+P 6400 2850
+AR Path="/5CE12F3D" Ref="Q?"  Part="1"
+AR Path="/5C753B69/5CE12F3D" Ref="Q10"  Part="1"
+F 0 "Q10" V 6743 2850 50  0000 C CNN
+F 1 "Q_PMOS_GSD" V 6652 2850 50  0000 C CNN
+F 2 "" H 6600 2950 50  0001 C CNN
+F 3 "~" H 6400 2850 50  0001 C CNN
+	1    6400 2850
+	0    1    -1   0
+$EndComp
+Connection ~ 6400 3050
 $EndSCHEMATC

Commit message: ADD: started routing
Parts:
- Q10: footprint (none) -> Package_TO_SOT_SMD:SOT-23
Changed lines of the file:
@@
 F 0 "Q10" V 6743 2850 50  0000 C CNN
 F 1 "Q_PMOS_GSD" V 6652 2850 50  0000 C CNN
-F 2 "" H 6600 2950 50  0001 C CNN
+F 2 "Package_TO_SOT_SMD:SOT-23" H 6600 2950 50  0001 C CNN
 F 3 "~" H 6400 2850 50  0001 C CNN
 	1    6400 2850
